File: PCB/Strojni_posuv/Strojni_posuv.kicad_pcb (KiCad board)
At the start: 2 copper layers, 170 x 80 mm, 169 parts, among them IC1 TB6600HG, J1 Conn_01x20_Pin, J10 Button_right_A, J11 Button_left_fast_A, J12 Button_right_fast_A, J13 Button_left_fast_B, J14 Button_right_fast_B, J2 Button_power_A, J3 OUT1, J4 OUT2, J5 POWER, J6 Button_power_B, J7 Button_left_A, J8 Button_left_B, J9 Button_right_A, Q1 BSS138, Q2 BSS138, Q3 BSS138, Q4 BSS138, Q5 BSS138, Q6 BSS138, Q7 BC847, SW2 SW_DPST_x2, SW3 SW_DPST_x2, SW4 SW_SPDT, SW5 RotaryEncoder_Switch, U1 STM32F103RBTx, U10 74AHCT1G125, U11 74AHCT1G125, U12 74AHCT1G125, U13 74AHCT1G125, U14 74AHCT1G125, U3 6N137, U5 6N137, U6 PC817, U7 74HC14, U8 TPS62822DLC, U9 74AHCT1G125, Y1 16MHz

Commit message: Revision 0
The PCB is done
Parts:
- added G***: LOGO, LOGO, F.Cu at (213.3, 45.7)
- added J15: STLINK, Connector_PinSocket_2.54mm:PinSocket_1x06_P2.54mm_Vertical, F.Cu at (159.2, 79.7)
- R46: value 10k -> 10K
- moved R2 9.08 mm to (111.2, 70.2), turned to 180 degrees
- moved J3 8.00 mm to (72.2, 100.5)
- moved J4 8.00 mm to (64.2, 100.5)
- moved C10 6.67 mm to (111.2, 72.2), turned to 180 degrees
- moved C26 6.23 mm to (94.2, 106.2), turned to 180 degrees
- moved C28 5.26 mm to (79.2, 95.0)
- moved D4 2.20 mm to (64.8, 96.9)
- moved R16 1.56 mm to (70.4, 97.0)
- moved J13 1.40 mm to (190.6, 36.9)
- moved J11 1.30 mm to (190.6, 41.8)
- moved R38 1.27 mm to (92.0, 103.5)
- moved U3 1.27 mm to (99.8, 100.1)
- moved C2 0.78 mm to (186.6, 78.0)
- moved CLK_END6 0.73 mm to (69.2, 63.3)
- moved R39 0.65 mm to (81.2, 59.3)
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Connections:
- C11 pad 2: Button_prec -> Button_conf
- R4 pad 2: Button_prec -> Button_conf
- R5 pad 2: Button_prec -> Button_conf
- U1 pad 46: unconnected-(U1-PA13-Pad46) -> /SWDIO
- U1 pad 49: unconnected-(U1-PA14-Pad49) -> /SWCLK
Routing:
- net +5V: track 0.00 -> 472.1 mm, vias 0 -> 9
- net +3.3V: track 0.00 -> 411.0 mm, vias 0 -> 13
- net Net-(D2-RK): track 0.00 -> 174.4 mm, vias 0 -> 1
- net Net-(D2-GK): track 0.00 -> 165.6 mm, vias 0 -> 1
- net Net-(D2-BK): track 0.00 -> 157.0 mm, vias 0 -> 1
- net M3: track 0.00 -> 133.6 mm, vias 0 -> 1
- net M1: track 0.00 -> 131.8 mm, vias 0 -> 1
- net M2: track 0.00 -> 114.5 mm, vias 0 -> 3
- net +48V: track 0.00 -> 109.6 mm, vias 0 -> 3
- net LTC: track 0.00 -> 102.8 mm, vias 0 -> 3
- net CLK: track 0.00 -> 95.9 mm, vias 0 -> 2
- net Enc_CLK: track 0.00 -> 86.9 mm, vias 0 -> 2
- net Button_encoder: track 0.00 -> 81.8 mm, vias 0 -> 2
- net Enc_DT: track 0.00 -> 80.4 mm
- net Button_conf: track 0.00 -> 79.3 mm, vias 0 -> 2
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Other:
- board text added: "HO HO"
- board text added: "JLCJLCJLCJLC"
- board text added: "Rev.0 251102"
