File: PCB/Strojni_posuv/Strojni_posuv.kicad_pcb (KiCad board)
At the start: 2 copper layers, 170 x 80 mm, 171 parts, among them IC1 TB6600HG, J1 Conn_01x20_Pin, J10 Button_right_A, J11 Button_left_fast_A, J12 Button_right_fast_A, J13 Button_left_fast_B, J14 Button_right_fast_B, J15 Conn_01x06_Socket, J2 Button_power_A, J3 OUT1, J4 OUT2, J5 POWER, J6 Button_power_B, J7 Button_left_A, J8 Button_left_B, J9 Button_right_A, Q1 BSS138, Q2 BSS138, Q3 BSS138, Q4 BSS138, Q5 BSS138, Q6 BSS138, Q7 BC847, SW2 SW_DPST_x2, SW3 SW_DPST_x2, SW4 SW_SPDT, SW5 RotaryEncoder_Switch, U1 STM32F103RBTx, U10 74AHCT1G125, U11 74AHCT1G125, U12 74AHCT1G125, U13 74AHCT1G125, U14 74AHCT1G125, U3 6N137, U5 6N137, U6 PC817, U7 74HC14, U8 TPS62822DLC, U9 74AHCT1G125, Y1 16MHz

Commit message: Starting new Revision 1
addressing some problems and mistakes
Parts:
- removed C26, C27: 100n, Capacitor_SMD:C_0603_1608Metric
- removed CLK_END6, DIR_END6: ~, TestPoint:TestPoint_Pad_D1.0mm
- removed D2: LED_RGBA, LED_THT:LED_D5.0mm-4_RGB_Wide_Pins
- removed J10: Button_right_A, Connector_Pin:Pin_D1.3mm_L11.3mm_W2.8mm_Flat
- removed J12: Button_right_fast_A, Connector_Pin:Pin_D1.3mm_L11.3mm_W2.8mm_Flat
- removed J13: Button_left_fast_B, Connector_Pin:Pin_D1.3mm_L11.3mm_W2.8mm_Flat
- removed J14: Button_right_fast_B, Connector_Pin:Pin_D1.3mm_L11.3mm_W2.8mm_Flat
- removed J8: Button_left_B, Connector_Pin:Pin_D1.3mm_L11.3mm_W2.8mm_Flat
- removed JP10, JP12, JP14, JP2, JP3, JP4, JP6, JP8: SolderJumper_2_Bridged, Jumper:SolderJumper-2_P1.3mm_Bridged_RoundedPad1.0x1.5mm
- removed JP11, JP13, JP15, JP5, JP7, JP9: SolderJumper_2_Open, Jumper:SolderJumper-2_P1.3mm_Open_RoundedPad1.0x1.5mm
- removed R38, R39, R40, R42: 4.7K, Resistor_SMD:R_0603_1608Metric
- removed RV1: 10K PRESET, Potentiometer_SMD:Potentiometer_Bourns_TC33X_Vertical
- removed U10, U11, U12, U13, U14, U9: 74AHCT1G125, Package_TO_SOT_SMD:SOT-353_SC-70-5
- removed U3, U5: 6N137, Package_SO:SOP-8_6.605x9.655mm_P2.54mm
- removed U6: PC817, Package_DIP:DIP-4_W8.89mm_SMDSocket_LongPads
- added D6: LED_BAGR, LED_THT:LED_D5.0mm-4_RGB_Wide_Pins, F.Cu at (79.3, 103.0)
- added J16: Buttons_fastR, Connector_JST:JST_XH_B2B-XH-A_1x02_P2.50mm_Vertical, F.Cu at (229.7, 46.8)
- added SW1: SW_SPDT_MSM, Button_Switch_THT:SW_CK_JS202011CQN_DPDT_Straight, F.Cu at (229.0, 38.7)
- C31: footprint Capacitor_SMD:C_0603_1608Metric -> Capacitor_SMD:C_0805_2012Metric
- C5: footprint Capacitor_SMD:C_0805_2012Metric -> Capacitor_SMD:C_0603_1608Metric
- J11: value Button_left_fast_A -> Button_fastL; footprint Connector_Pin:Pin_D1.3mm_L11.3mm_W2.8mm_Flat -> Connector_JST:JST_XH_B2B-XH-A_1x02_P2.50mm_Vertical
- J7: value Button_left_A -> Button_maxL; footprint Connector_Pin:Pin_D1.3mm_L11.3mm_W2.8mm_Flat -> Connector_JST:JST_XH_B2B-XH-A_1x02_P2.50mm_Vertical
- J9: value Button_right_A -> Button_maxR; footprint Connector_Pin:Pin_D1.3mm_L11.3mm_W2.8mm_Flat -> Connector_JST:JST_XH_B2B-XH-A_1x02_P2.50mm_Vertical
- R1, R10, R11, R12, R13, R14, R15, R16, R17, R18, R2, R25, R26, R27, R28, R29, R3, R30, R31, R32, R33, R34, R35, R36, R37, R4, R41, R43, R44, R45, R46, R47, R48, R49, R5, R50, R51, R52, R53, R54, R55, R56, R6, R7, R8, R9: footprint Resistor_SMD:R_0603_1608Metric -> Resistor_SMD:R_0805_2012Metric
- R19: value 680m -> 10K; footprint Resistor_SMD:R_1206_3216Metric -> Resistor_SMD:R_0805_2012Metric
- R20, R21, R23, R24: value 680m -> 330m; footprint Resistor_SMD:R_1206_3216Metric -> Resistor_THT:R_Axial_DIN0922_L20.0mm_D9.0mm_P30.48mm_Horizontal
- R22: value 680m -> 16.5K; footprint Resistor_SMD:R_1206_3216Metric -> Resistor_SMD:R_0805_2012Metric
- moved R21 64.4 mm to (19.0, 87.7)
- moved R23 55.8 mm to (30.0, 87.7)
- moved R24 47.5 mm to (41.0, 88.2)
Connections:
- C25 pad 1: Net-(IC1-VREG) -> +5V
- IC1 pad 18_1: /Motor_driver/ENB -> +5V
- IC1 pad 21: /Motor_driver/CLK_L -> CLK
- IC1 pad 22_1: /Motor_driver/DIR_L -> DIR
- IC1 pad 24_1: Net-(IC1-VREG) -> +5V
- Q1 pad 2: Net-(JP11-B) -> M1_STM
- Q2 pad 2: Net-(JP13-B) -> M3_STM
- Q3 pad 2: Net-(JP9-B) -> LTC_STM
- Q4 pad 2: Net-(JP15-B) -> M2_STM
- Q5 pad 2: Net-(JP7-B) -> STEP_STM
- Q6 pad 2: Net-(JP5-B) -> DIR_STM
- R19 pad 1: Net-(IC1-NFB) -> GND
- R19 pad 2: GND -> Net-(IC1-VREF)
- R22 pad 1: GND -> +5V
- R22 pad 2: Net-(IC1-NFA) -> Net-(IC1-VREF)
- R25 pad 1: Net-(JP11-B) -> M1_STM
- R27 pad 1: Net-(JP15-B) -> M2_STM
- R29 pad 1: Net-(JP13-B) -> M3_STM
- R31 pad 1: Net-(JP9-B) -> LTC_STM
- R34 pad 1: Net-(JP7-B) -> STEP_STM
- R36 pad 1: Net-(JP5-B) -> DIR_STM
- U1 pad 43: Enc_CLK -> unconnected-(U1-PA10-Pad43)
- U1 pad 44: Enc_DT -> unconnected-(U1-PA11-Pad44)
- U1 pad 50: unconnected-(U1-PA15-Pad50) -> Enc_CLK
- U1 pad 55: unconnected-(U1-PB3-Pad55) -> Enc_DT
Routing:
- net +5V: track 472.9 -> 562.1 mm, vias 9 -> 11
- net /Motor_driver/ENB: track 74.4 -> 0.00 mm, vias 1 -> 0
- net DIR: track 64.1 -> 120.8 mm, vias 0 -> 3
- net /Motor_driver/DIR_L: track 56.7 -> 0.00 mm, vias 3 -> 0
- net (no net): track 0.00 -> 44.3 mm
- net Net-(IC1-VREG): track 14.8 -> 0.00 mm, vias 1 -> 0
- net Net-(R42-Pad1): track 12.3 -> 0.00 mm
- net Net-(JP5-B): track 8.27 -> 0.00 mm
- net DIR_STM: track 63.5 -> 71.8 mm
- net Net-(JP7-B): track 8.26 -> 0.00 mm
- net STEP_STM: track 58.8 -> 67.1 mm
- net Net-(JP9-B): track 8.23 -> 0.00 mm
- net LTC_STM: track 71.0 -> 79.2 mm
- net M3_STM: track 71.6 -> 79.8 mm
- net Net-(JP13-B): track 8.20 -> 0.00 mm
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Other:
- board size 170 x 80 mm -> 210 x 80 mm

Commit message: Resolving problems from list
Parts:
- removed C12: 100n, Capacitor_SMD:C_0603_1608Metric
- removed J11: Button_fastL, Connector_JST:JST_XH_B2B-XH-A_1x02_P2.50mm_Vertical
- removed J16: Buttons_fastR, Connector_JST:JST_XH_B2B-XH-A_1x02_P2.50mm_Vertical
- removed R6: 16.5K, Resistor_SMD:R_0805_2012Metric
- removed R8: 470, Resistor_SMD:R_0805_2012Metric
- removed SW3: SW_DPST_x2, Button_Switch_THT:SW_PUSH_6mm
- added SW6: Emergency_stop, Emergency:Emergency_stop, F.Cu at (264.5, 98.0)
- SW1: footprint Button_Switch_THT:SW_CK_JS202011CQN_DPDT_Straight -> ON_Off_ON:on_off_on
- moved SW5 130.3 mm to (228.2, 90.0)
- moved SW1 127.8 mm to (105.5, 71.5), turned to 90 degrees
- moved SW2 122.1 mm to (218.5, 74.0)
- moved R21 75.9 mm to (66.5, 147.0)
- moved R23 75.9 mm to (77.5, 147.0)
- moved R24 75.9 mm to (88.5, 147.4)
- moved SW4 23.4 mm to (231.9, 76.5)
Connections:
- J6 pad 1: GND -> Net-(J6-Pin_1)
- R51 pad 1: Net-(J11-Pin_1) -> Net-(SW1-4)
- R52 pad 1: Net-(J16-Pin_1) -> Net-(R52-Pad1)
- SW1 pad 1: unconnected-(SW1-Pad1) -> Net-(R52-Pad1)
- SW1 pad 2: unconnected-(SW1-3-Pad2) -> +3.3V
- SW1 pad 3: unconnected-(SW1-4-Pad3) -> Net-(SW1-4)
- U1 pad 10: Button_gen_stop -> unconnected-(U1-PC2-Pad10)
Routing:
- net unconnected-(U1-PC2-Pad10): track 0.00 -> 34.5 mm, vias 0 -> 2
- net Button_gen_stop: track 34.5 -> 0.00 mm, vias 2 -> 0
- net (no net): track 44.3 -> 53.6 mm
- net Net-(SW3A-A): track 9.31 -> 0.00 mm
- net Net-(SW1-4): track 0.00 -> 5.19 mm
- net Net-(J11-Pin_1): track 5.19 -> 0.00 mm
- net Net-(R52-Pad1): track 0.00 -> 4.34 mm
- net Net-(J16-Pin_1): track 4.34 -> 0.00 mm
Other:
- board size 210 x 80 mm -> 227 x 80 mm

Commit message: Schema done?
I think that I have functional schema, but it needs a check
Parts:
- removed J15: Conn_01x06_Socket, Connector_PinSocket_2.54mm:PinSocket_1x06_P2.54mm_Vertical
- added EN1: ~, TestPoint:TestPoint_Pad_D1.0mm, F.Cu at (130.2, 120.3)
- added J10: Conn_01x05_Socket, Connector_JST:JST_PH_B5B-PH-K_1x05_P2.00mm_Vertical, F.Cu at (243.5, 63.2)
- added LEN1: ~, TestPoint:TestPoint_Pad_D1.0mm, F.Cu at (130.2, 123.4)
- added LRST1: ~, TestPoint:TestPoint_Pad_D1.0mm, F.Cu at (130.2, 126.5)
- added Q8: BSS138, Package_TO_SOT_SMD:SOT-23, F.Cu at (139.1, 121.1)
- added Q9: BSS138, Package_TO_SOT_SMD:SOT-23, F.Cu at (139.1, 125.8)
- added R38: 10K, Resistor_SMD:R_0805_2012Metric, F.Cu at (134.4, 126.1)
- added R39: 10K, Resistor_SMD:R_0805_2012Metric, F.Cu at (134.4, 129.1)
- added R6: 10K, Resistor_SMD:R_0805_2012Metric, F.Cu at (134.4, 120.2)
- added R8: 10K, Resistor_SMD:R_0805_2012Metric, F.Cu at (134.4, 123.2)
- added RST1: ~, TestPoint:TestPoint_Pad_D1.0mm, F.Cu at (130.2, 129.5)
- moved SW6 55.0 mm to (264.8, 43.0)
- moved SW4 9.02 mm to (240.8, 74.8)
Connections:
- IC1 pad 18_1: +5V -> EN
- IC1 pad 19: +5V -> RST
- U1 pad 16: unconnected-(U1-PA2-Pad16) -> PA2
- U1 pad 33: unconnected-(U1-PB12-Pad33) -> Enable
- U1 pad 35: unconnected-(U1-PB14-Pad35) -> Reset
- U1 pad 42: unconnected-(U1-PA9-Pad42) -> PA9
- U1 pad 56: unconnected-(U1-PB4-Pad56) -> PB4
- U1 pad 57: unconnected-(U1-PB5-Pad57) -> PB5
Routing:
- net +5V: track 562.1 -> 487.7 mm, vias 11 -> 10
- net EN: track 0.00 -> 74.4 mm, vias 0 -> 1

Commit message: PCB done?
I did all the routing and component placement on PCB
Parts:
- removed D1: LED, LED_SMD:LED_0603_1608Metric
- removed JP1: SolderJumper_2_Open, Jumper:SolderJumper-2_P1.3mm_Open_TrianglePad1.0x1.5mm
- removed R45: 470, Resistor_SMD:R_0805_2012Metric
- removed SW2: SW_DPST_x2, Button_Switch_THT:SW_PUSH_6mm
- added J11: Volne_IO_Power, TerminalBlock:TerminalBlock_Xinya_XY308-2.54-3P_1x03_P2.54mm_Horizontal, B.Cu at (228.9, 104.0)
- added J12: Button_conf, Connector_JST:JST_XH_B2B-XH-A_1x02_P2.50mm_Vertical, B.Cu at (226.0, 81.0)
- added J8: Volne_IO, TerminalBlock:TerminalBlock_Xinya_XY308-2.54-3P_1x03_P2.54mm_Horizontal, B.Cu at (218.9, 104.0)
- J10, J7, J9: moved to B.Cu
- J3, J4: footprint Connector_PinSocket_2.54mm:PinSocket_1x02_P2.54mm_Vertical -> TerminalBlock_Phoenix:TerminalBlock_Phoenix_MKDS-1,5-2-5.08_1x02_P5.08mm_Horizontal; moved to B.Cu
- moved SW6 205.8 mm to (59.0, 42.0), turned to 90 degrees
- moved R52 127.8 mm to (75.0, 69.5)
- moved R50 127.2 mm to (74.0, 74.0), turned to 90 degrees
- moved C34 125.4 mm to (76.5, 74.0), turned to 90 degrees
- moved R5 124.6 mm to (231.5, 81.9), turned to -90 degrees
- moved R4 123.5 mm to (234.0, 86.6), turned to 90 degrees
- moved C11 121.0 mm to (231.5, 86.5), turned to 90 degrees
- moved R47 107.3 mm to (214.5, 81.5)
- moved R49 106.9 mm to (83.5, 78.2)
- moved C33 106.5 mm to (86.0, 81.0), turned to 90 degrees
- moved R51 105.2 mm to (88.5, 78.2), turned to 180 degrees
- moved C10 101.1 mm to (211.5, 59.0)
- moved R3 100.8 mm to (207.4, 55.5), turned to 0 degrees
- moved R48 100.2 mm to (207.4, 81.5), turned to 0 degrees
- moved R2 96.9 mm to (207.5, 59.0), turned to 0 degrees
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Connections:
- LEN1 pad 1: /Motor_driver/EN1 -> Enable
- LRST1 pad 1: /Motor_driver/RST1 -> Reset
- Q8 pad 2: /Motor_driver/EN1 -> Enable
- Q9 pad 2: /Motor_driver/RST1 -> Reset
- R38 pad 1: /Motor_driver/RST1 -> Reset
- R6 pad 1: /Motor_driver/EN1 -> Enable
- U1 pad 14: ADC1 -> PA0
- U1 pad 15: ADC2 -> PA1
- U1 pad 17: unconnected-(U1-PA3-Pad17) -> PA3
- U1 pad 42: PA9 -> unconnected-(U1-PA9-Pad42)
- U1 pad 56: PB4 -> unconnected-(U1-PB4-Pad56)
- U1 pad 57: PB5 -> unconnected-(U1-PB5-Pad57)
Routing:
- net +5V: track 487.7 -> 309.9 mm, vias 10 -> 12
- net +3.3V: track 411.0 -> 527.7 mm, vias 13 -> 9
- net RST: track 0.00 -> 94.9 mm, vias 0 -> 2
- net PA3: track 0.00 -> 69.4 mm, vias 0 -> 1
- net Button_right_fast: track 42.4 -> 107.9 mm, vias 0 -> 2
- net M1_STM: track 85.2 -> 21.4 mm, vias 2 -> 0
- net PA2: track 0.00 -> 63.5 mm, vias 0 -> 1
- net Button_right_max: track 48.6 -> 111.8 mm
- net PA1: track 0.00 -> 61.9 mm, vias 0 -> 1
- net Left: track 32.9 -> 93.3 mm, vias 0 -> 2
- net PA0: track 0.00 -> 59.7 mm, vias 0 -> 1
- net M2_STM: track 83.0 -> 29.2 mm
- net (no net): track 53.6 -> 0.00 mm
- net Button_left_max: track 42.0 -> 91.7 mm, vias 2 -> 4
- net LTC_STM: track 79.2 -> 30.1 mm, vias 2 -> 0
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Other:
- outline, holes or cut-outs redrawn
- board text added: "Rev.1 251102"
- board text removed: "HO HO"
- board text removed: "Rev.0 251102"
