File: PCB/Strojni_posuv/power.kicad_sch (KiCad schematic)
At the start: 29 parts, among them J2 Button_power_A, J5 POWER, J6 Button_power_B, U4 MIC5365-3.3YC5, U8 TPS62822DLC

Commit message: Revision 0 - final
I send this files to JLCPCB
Parts:
- removed C18, C19: 22u, Capacitor_SMD:C_2220_5750Metric, symbol Device:C
- added C18, C19: 22u, Capacitor_SMD:CP_Elec_6.3x5.4, symbol Device:C_Polarized
Connections:
- net +48V: now also C18.1, C19.1
- net GND: now also C18.2, C19.2
Changed lines of the file:
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@@
 	)
 	(symbol
+		(lib_id "Device:C_Polarized")
+		(at 30.48 48.26 0)
+		(unit 1)
+		(exclude_from_sim no)
+		(in_bom yes)
+		(on_board yes)
+		(dnp no)
+		(fields_autoplaced yes)
+		(property "Reference" "C18"
+			(at 34.29 46.1009 0)
+			(effects
+				(font
+					(size 1.27 1.27)
+				)
+				(justify left)
+			)
+		)
+		(property "Value" "22u"
+			(at 34.29 48.6409 0)
+			(effects
+				(font
+					(size 1.27 1.27)
+				)
+				(justify left)
+			)
+		)
+		(property "Footprint" "Capacitor_SMD:CP_Elec_6.3x5.4"
+			(at 31.4452 52.07 0)
+			(effects
+				(font
+					(size 1.27 1.27)
+				)
+				(hide yes)
+			)
+		)
+		(property "Datasheet" "~"
+			(at 30.48 48.26 0)
+			(effects
+				(font
+					(size 1.27 1.27)
+				)
+				(hide yes)
+			)
+		)
+		(property "Description" "Polarized capacitor"
+			(at 30.48 48.26 0)
+			(effects
+				(font
+					(size 1.27 1.27)
+				)
+				(hide yes)
+			)
+		)
+		(property "LCSC" "C2836438"
+			(at 30.48 48.26 0)
+			(effects
+				(font
+					(size 1.27 1.27)
+				)
+				(hide yes)
+			)
+		)
+		(pin "2"
+		)
+		(pin "1"
+		)
+		(instances
+			(project ""
+				(path "/36664f97-4753-4126-9e35-a8ab7ac5ffb4/ee0b1210-eaee-41ba-b593-299cdfd1f985"
+					(reference "C18")
+					(unit 1)
+				)
+			)
+		)
+	)
+	(symbol
 		(lib_id "Device:C")
 		(at 161.29 179.07 180)
@@
 	)
 	(symbol
-		(lib_id "power:GND")
-		(at 30.48 54.61 0)
+		(lib_id "Device:C_Polarized")
+		(at 41.91 48.26 0)
 		(unit 1)
 		(exclude_from_sim no)
@@
 		(dnp no)
 		(fields_autoplaced yes)
-		(property "Reference" "#PWR027"
-			(at 30.48 60.96 0)
+		(property "Reference" "C19"
+			(at 45.72 46.1009 0)
 			(effects
 				(font
 					(size 1.27 1.27)
 				)
-				(hide yes)
+				(justify left)
 			)
 		)
-		(property "Value" "GND"
-			(at 30.48 59.69 0)
+		(property "Value" "22u"
+			(at 45.72 48.6409 0)
+			(effects
+				(font
+					(size 1.27 1.27)
+				)
+				(justify left)
+			)
+		)
+		(property "Footprint" "Capacitor_SMD:CP_Elec_6.3x5.4"
+			(at 42.8752 52.07 0)
 			(effects
 				(font
@@
 			)
 		)
-		(property "Footprint" ""
-			(at 30.48 54.61 0)
+		(property "Datasheet" "~"
+			(at 41.91 48.26 0)
 			(effects
 				(font
@@
 			)
 		)
-		(property "Datasheet" ""
-			(at 30.48 54.61 0)
+		(property "Description" "Polarized capacitor"
+			(at 41.91 48.26 0)
 			(effects
 				(font
@@
 			)
 		)
-		(property "Description" ""
-			(at 30.48 54.61 0)
+		(property "LCSC" "C2836438"
+			(at 41.91 48.26 0)
 			(effects
 				(font
@@
 			)
 		)
+		(pin "2"
+		)
 		(pin "1"
 		)
@@
 			(project "Strojni_posuv"
 				(path "/36664f97-4753-4126-9e35-a8ab7ac5ffb4/ee0b1210-eaee-41ba-b593-299cdfd1f985"
-					(reference "#PWR027")
+					(reference "C19")
 					(unit 1)
 				)
@@
 	)
 	(symbol
-		(lib_id "Device:R")
-		(at 118.11 71.12 180)
+		(lib_id "power:GND")
+		(at 30.48 54.61 0)
 		(unit 1)
 		(exclude_from_sim no)
@@
 		(on_board yes)
 		(dnp no)
-		(property "Reference" "R18"
-			(at 121.158 67.056 0)
-			(effects
-				(font
-					(size 1.27 1.27)
-				)
-			)
-		)
-		(property "Value" "240K"
-			(at 115.57 71.12 90)
-			(effects
-				(font
-					(size 1.27 1.27)
-				)
-			)
-		)
-		(property "Footprint" "Resistor_SMD:R_0603_1608Metric"
-			(at 119.888 71.12 90)
-			(effects
-				(font
-					(size 1.27 1.27)
-				)
-				(hide yes)
-			)
-		)
-		(property "Datasheet" "~"
-			(at 118.11 71.12 0)
+		(fields_autoplaced yes)
+		(property "Reference" "#PWR027"
+			(at 30.48 60.96 0)
 			(effects
 				(font
@@
 			)
 		)
-		(property "Description" ""
-			(at 118.11 71.12 0)
+		(property "Value" "GND"
+			(at 30.48 59.69 0)
 			(effects
 				(font
@@
 			)
 		)
-		(property "LCSC" "C4197"
-			(at 118.11 71.12 0)
+		(property "Footprint" ""
+			(at 30.48 54.61 0)
 			(effects
 				(font
@@
 			)
 		)
-		(property "Field5" ""
-			(at 118.11 71.12 0)
+		(property "Datasheet" ""
+			(at 30.48 54.61 0)
 			(effects
 				(font
@@
 			)
 		)
-		(property "LSCS" ""
-			(at 118.11 71.12 0)
+		(property "Description" ""
+			(at 30.48 54.61 0)
 			(effects
 				(font
@@
 		(pin "1"
 		)
-		(pin "2"
-		)
 		(instances
 			(project "Strojni_posuv"
 				(path "/36664f97-4753-4126-9e35-a8ab7ac5ffb4/ee0b1210-eaee-41ba-b593-299cdfd1f985"
-					(reference "R18")
+					(reference "#PWR027")
 					(unit 1)
 				)
@@
 	)
 	(symbol
-		(lib_id "Device:C")
-		(at 41.91 48.26 0)
+		(lib_id "Device:R")
+		(at 118.11 71.12 180)
 		(unit 1)
 		(exclude_from_sim no)
@@
 		(on_board yes)
 		(dnp no)
-		(fields_autoplaced yes)
-		(property "Reference" "C19"
-			(at 45.72 46.9899 0)
+		(property "Reference" "R18"
+			(at 121.158 67.056 0)
 			(effects
 				(font
 					(size 1.27 1.27)
 				)
-				(justify left)
 			)
 		)
-		(property "Value" "22u"
-			(at 45.72 49.5299 0)
+		(property "Value" "240K"
+			(at 115.57 71.12 90)
 			(effects
 				(font
 					(size 1.27 1.27)
 				)
-				(justify left)
 			)
 		)
-		(property "Footprint" "Capacitor_SMD:C_2220_5750Metric"
-			(at 42.8752 52.07 0)
+		(property "Footprint" "Resistor_SMD:R_0603_1608Metric"
+			(at 119.888 71.12 90)
 			(effects
 				(font
@@
 		)
 		(property "Datasheet" "~"
-			(at 41.91 48.26 0)
+			(at 118.11 71.12 0)
 			(effects
 				(font
@@
 			)
 		)
-		(property "Description" "Unpolarized capacitor"
-			(at 41.91 48.26 0)
+		(property "Description" ""
+			(at 118.11 71.12 0)
 			(effects
 				(font
@@
 			)
 		)
-		(property "LCSC" "C784103"
-			(at 41.91 48.26 0)
+		(property "LCSC" "C4197"
+			(at 118.11 71.12 0)
 			(effects
 				(font
@@
 		)
 		(property "Field5" ""
-			(at 41.91 48.26 0)
+			(at 118.11 71.12 0)
 			(effects
 				(font
@@
 		)
 		(property "LSCS" ""
-			(at 41.91 48.26 0)
+			(at 118.11 71.12 0)
 			(effects
 				(font
@@
 			)
 		)
-		(pin "2"
-		)
 		(pin "1"
 		)
+		(pin "2"
+		)
 		(instances
 			(project "Strojni_posuv"
 				(path "/36664f97-4753-4126-9e35-a8ab7ac5ffb4/ee0b1210-eaee-41ba-b593-299cdfd1f985"
-					(reference "C19")
+					(reference "R18")
 					(unit 1)
 				)
@@
 					(unit 1)
 				)
-			)
-		)
-	)
-	(symbol
-		(lib_id "Device:C")
-		(at 30.48 48.26 0)
-		(unit 1)
-		(exclude_from_sim no)
-		(in_bom yes)
-		(on_board yes)
-		(dnp no)
-		(fields_autoplaced yes)
-		(property "Reference" "C18"
-			(at 34.29 46.9899 0)
-			(effects
-				(font
-					(size 1.27 1.27)
-				)
-				(justify left)
-			)
-		)
-		(property "Value" "22u"
-			(at 34.29 49.5299 0)
-			(effects
-				(font
-					(size 1.27 1.27)
-				)
-				(justify left)
-			)
-		)
-		(property "Footprint" "Capacitor_SMD:C_2220_5750Metric"
-			(at 31.4452 52.07 0)
-			(effects
-				(font
-					(size 1.27 1.27)
-				)
-				(hide yes)
-			)
-		)
-		(property "Datasheet" "~"
-			(at 30.48 48.26 0)
-			(effects
-				(font
-					(size 1.27 1.27)
-				)
-				(hide yes)
-			)
-		)
-		(property "Description" "Unpolarized capacitor"
-			(at 30.48 48.26 0)
-			(effects
-				(font
-					(size 1.27 1.27)
-				)
-				(hide yes)
-			)
-		)
-		(property "LCSC" "C784103"
-			(at 30.48 48.26 0)
-			(effects
-				(font
-					(size 1.27 1.27)
-				)
-				(hide yes)
-			)
-		)
-		(property "Field5" ""
-			(at 30.48 48.26 0)
-			(effects
-				(font
-					(size 1.27 1.27)
-				)
-				(hide yes)
-			)
-		)
-		(property "LSCS" ""
-			(at 30.48 48.26 0)
-			(effects
-				(font
-					(size 1.27 1.27)
-				)
-				(hide yes)
-			)
-		)
-		(pin "2"
-		)
-		(pin "1"
-		)
-		(instances
-			(project ""
-				(path "/36664f97-4753-4126-9e35-a8ab7ac5ffb4/ee0b1210-eaee-41ba-b593-299cdfd1f985"
-					(reference "C18")
-					(unit 1)
-				)
