File: PCB/Strojni_posuv/power.kicad_sch (KiCad schematic)
At the start: 27 parts, among them J2 Button_power_A, J5 POWER, J6 Button_power_B, SW6 Emergency_stop, U4 MIC5365-3.3YC5, U8 TPS62822DLC

Commit message: Numpad + small changes
I added numpad and add some description to components
Parts:
- C31: LCSC C1705 -> C1779
- J2, J6, SW6: now not fitted
- R12: LCSC C23179 -> C17710
- R17, R46: LCSC C25804 -> C17414
- R18: LCSC C4197 -> C25824
- R44: LCSC C23058 -> C322483
