File: PCB/Strojni_posuv/motor_driver.kicad_sch (KiCad schematic)
At the start: 60 parts, among them IC1 TB6600HG, J3 OUT1, J4 OUT2, Q1 BSS138, Q2 BSS138, Q3 BSS138, Q4 BSS138, Q5 BSS138, Q6 BSS138, Q7 BC847, Q8 BSS138, Q9 BSS138, U7 74HC14

Commit message: Numpad + small changes
I added numpad and add some description to components
Parts:
- R16, R33, R43: LCSC C23179 -> C17710
- R19, R25, R26, R27, R28, R29, R30, R31, R32, R34, R35, R36, R37, R38, R39, R6, R8: LCSC C25804 -> C17414
- R20, R21, R23, R24: LCSC C19108 -> (none); now not fitted
- R22: LCSC C22812 -> C2930171
- R41: LCSC C23196 -> C17737
