File: PCB/Strojni_posuv/Strojni_posuv.kicad_sch (KiCad schematic)
At the start: 56 parts, among them J1 Conn_01x20_Pin, J10 Conn_01x05_Socket, J11 Volne_IO_Power, J12 Button_conf, J7 Button_maxL, J8 Volne_IO, J9 Button_maxR, SW1 SW_SPDT_MSM, SW4 SW_SPDT, SW5 RotaryEncoder_Switch, U1 STM32F103RBTx, Y1 16MHz

Commit message: Numpad + small changes
I added numpad and add some description to components
Parts:
- added Numpad1: Conn_01x08_Socket, Connector_PinSocket_2.54mm:PinSocket_1x08_P2.54mm_Vertical, symbol Connector:Conn_01x08_Socket
- C5: LCSC C15850 -> C1691
- J12, J7, J9, SW1, SW4, SW5: now not fitted
- R1, R47, R48: LCSC C25804 -> C17414
- R10, R2, R4, R49, R50, R53, R55, R7: LCSC C22812 -> C2930171
- R11, R13, R14, R15, R3, R5, R51, R52, R54, R56, R9: LCSC C23179 -> C17710
Connections:
- net NumPB11: now reaches U1.30 (PB11)
- net NumPB11: now also Numpad1.7 (Pin_7)
- net NumPB13: now reaches U1.34 (PB13)
- net NumPB13: now also Numpad1.6 (Pin_6)
- net NumPB15: now reaches U1.36 (PB15)
- net NumPB15: now also Numpad1.5 (Pin_5)
- net NumPA9: now reaches U1.42 (PA9)
- net NumPA9: now also Numpad1.8 (Pin_8)
- net NumPA10: now reaches U1.43 (PA10)
- net NumPA10: now also Numpad1.4 (Pin_4)
- net NumPA11: now reaches U1.44 (PA11)
- net NumPA11: now also Numpad1.3 (Pin_3)
- net NumPA12: now reaches U1.45 (PA12)
- net NumPA12: now also Numpad1.2 (Pin_2)
- net NumPD2: now reaches U1.54 (PD2)
- net NumPD2: now also Numpad1.1 (Pin_1)
